File: NeoPLC.kicad_sch (KiCad schematic)
At the start: 0 parts

Commit message: DI-8 şema ve PCB taslağı: platform kararları kilitlendi, çekirdek/saha yerleşimi GitHub’da.
Birkaç saatlik stabil anlarda origin’e push kuralı eklendi; yerel KiCAD geçmişi ve Konnect önizlemeleri commit dışı bırakıldı.

Co-authored-by: Cursor <cursoragent@cursor.com>
Other:
- added sheet DI Field (di_field.kicad_sch)
- added sheet Node Core (node_core.kicad_sch)
- note added: "First node, platform bring-up. Sheet 1: Node Core (backplane, 5V-3V3, MCU, RS-485, SWD). Sheet 2: DI Field (8ch isolated)."
- note added: "NeoPLC DI-8 | Rev 0.1 | 2026-09-17"
Changed lines of the file:
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@@
 	(generator_version "10.0")
 	(paper "A4")
+	(wire
+		(pts
+			(xy 140.97 40.64)
+			(xy 157.48 40.64)
+		)
+	)
+	(wire
+		(pts
+			(xy 140.97 43.18)
+			(xy 157.48 43.18)
+		)
+	)
+	(wire
+		(pts
+			(xy 140.97 45.72)
+			(xy 157.48 45.72)
+		)
+	)
+	(wire
+		(pts
+			(xy 140.97 48.26)
+			(xy 157.48 48.26)
+		)
+	)
+	(wire
+		(pts
+			(xy 140.97 50.8)
+			(xy 157.48 50.8)
+		)
+	)
+	(wire
+		(pts
+			(xy 140.97 53.34)
+			(xy 157.48 53.34)
+		)
+	)
+	(wire
+		(pts
+			(xy 140.97 55.88)
+			(xy 157.48 55.88)
+		)
+	)
+	(wire
+		(pts
+			(xy 140.97 58.42)
+			(xy 157.48 58.42)
+		)
+	)
+	(text "NeoPLC DI-8  |  Rev 0.1  |  2026-09-17"
+		(at 30.48 25.4 0)
+		(effects
+			(font
+				(size 2.54 2.54)
+				(bold yes)
+			)
+			(justify left bottom)
+		)
+	)
+	(text "First node, platform bring-up. Sheet 1: Node Core (backplane, 5V-3V3, MCU, RS-485, SWD). Sheet 2: DI Field (8ch isolated)."
+		(at 30.48 30.48 0)
+		(effects
+			(font
+				(size 1.27 1.27)
+			)
+			(justify left bottom)
+		)
+	)
+	(sheet
+		(at 30.48 38.1)
+		(size 110.49 90)
+		(fields_autoplaced)
+		(stroke
+			(width 0.1524)
+			(type solid)
+		)
+		(fill
+			(color 0 0 0 0.0)
+		)
+		(property "Sheetname" "Node Core"
+			(at 30.48 37.465 0)
+			(effects
+				(font
+					(size 1.27 1.27)
+				)
+				(justify left bottom)
+			)
+		)
+		(property "Sheetfile" "node_core.kicad_sch"
+			(at 30.48 128.73499999999999 0)
+			(effects
+				(font
+					(size 1.27 1.27)
+				)
+				(justify left top)
+			)
+		)
+		(pin "DI1" input
+			(at 140.97 40.64 0)
+		)
+		(pin "DI2" input
+			(at 140.97 43.18 0)
+		)
+		(pin "DI3" input
+			(at 140.97 45.72 0)
+		)
+		(pin "DI4" input
+			(at 140.97 48.26 0)
+		)
+		(pin "DI5" input
+			(at 140.97 50.8 0)
+		)
+		(pin "DI6" input
+			(at 140.97 53.34 0)
+		)
+		(pin "DI7" input
+			(at 140.97 55.88 0)
+		)
+		(pin "DI8" input
+			(at 140.97 58.42 0)
+		)
+		(instances
+			(project "NeoPLC"
+				(path "/c984adae-5495-4a3b-b0a6-3ee1775863dd"
+					(page "2")
+				)
+			)
+		)
+	)
+	(sheet
+		(at 157.48 38.1)
+		(size 110 90)
+		(fields_autoplaced)
+		(stroke
+			(width 0.1524)
+			(type solid)
+		)
+		(fill
+			(color 0 0 0 0.0)
+		)
+		(property "Sheetname" "DI Field"
+			(at 157.48 37.465 0)
+			(effects
+				(font
+					(size 1.27 1.27)
+				)
+				(justify left bottom)
+			)
+		)
+		(property "Sheetfile" "di_field.kicad_sch"
+			(at 157.48 128.73499999999999 0)
+			(effects
+				(font
+					(size 1.27 1.27)
+				)
+				(justify left top)
+			)
+		)
+		(pin "DI1" output
+			(at 157.48 40.64 180)
+		)
+		(pin "DI2" output
+			(at 157.48 43.18 180)
+		)
+		(pin "DI3" output
+			(at 157.48 45.72 180)
+		)
+		(pin "DI4" output
+			(at 157.48 48.26 180)
+		)
+		(pin "DI5" output
+			(at 157.48 50.8 180)
+		)
+		(pin "DI6" output
+			(at 157.48 53.34 180)
+		)
+		(pin "DI7" output
+			(at 157.48 55.88 180)
+		)
+		(pin "DI8" output
+			(at 157.48 58.42 180)
+		)
+		(instances
+			(project "NeoPLC"
+				(path "/c984adae-5495-4a3b-b0a6-3ee1775863dd"
+					(page "3")
+				)
+			)
+		)
+	)
 )
